File: NumPad/NumPad.kicad_sch (KiCad schematic)
At the start: 0 parts

Commit message: starting schematic drawing
Parts:
- added R1: R_Small_US, symbol Device:R_Small_US
- added U1: ATmega32U4-A, Package_QFP:TQFP-44_10x10mm_P0.8mm, symbol MCU_Microchip_ATmega:ATmega32U4-A
Connections:
- new net: R1.1, U1.33 (~{HWB}/PE2)
- new net +5V: U1.14 (VCC), U1.2 (UVCC), U1.24 (AVCC), U1.34 (VCC), U1.44 (AVCC)
- new net GND: R1.2, U1.15 (GND), U1.23 (GND), U1.35 (GND), U1.43 (GND), U1.5 (UGND)

Commit message: finished MCU schematic
Parts:
- added C1: 1μF, symbol Device:C_Small_US
- added C2, C3, C4: 0.1μF, symbol Device:C_Small_US
- added C5: 10μF, symbol Device:C_Small_US
- added C6, C7: 22pF, symbol Device:C_Small_US
- added R2, R3: 22, symbol Device:R_Small_US
- added R4: 10k, symbol Device:R_Small_US
- added SW1: SW_Push, symbol Switch:SW_Push
- added Y1: 16MHz, symbol Device:Crystal_GND24_Small
- R1: value R_Small_US -> 10k
Connections:
- net +5V: now also U1.7 (VBUS), C2.1, C3.1, C4.1, C5.1, R4.1
- net GND: now also C1.2, C2.2, C3.2, C4.2, C5.2, C6.1, C7.1, SW1.1, Y1.2, Y1.4
- net at U1.13 (~{RESET}): now also R4.2, SW1.2
- net at U1.16 (XTAL2): now also C7.2, Y1.3
- net at U1.17 (XTAL1): now also C6.2, Y1.1
- net at U1.3 (D-): now also R3.2
- net at U1.4 (D+): now also R2.2
- net at U1.6 (UCAP): now also C1.1
- new net D+: R2.1
- new net D-: R3.1
Other:
- moved on the sheet: R1

Commit message: updated connector to usb-C with only usb2.0 functionality
Used documentation from guide as well as dubious creations (https://dubiouscreations.com/2021/04/06/designing-with-usb-c-lessons-learned/)
Parts:
- added F2: 500mA, symbol Device:Polyfuse_Small
- added J1: USB_C_Receptacle_USB2.0_16P, symbol Connector:USB_C_Receptacle_USB2.0_16P
- added R5, R6: 5.1kΩ, symbol Device:R_Small_US
- R1, R4: value 10k -> 10kΩ
- R2, R3: value 22 -> 22Ω
Connections:
- net +5V: now also F2.2
- net D+: now also J1.A6 (D+), J1.B6 (D+)
- net D-: now also J1.A7 (D-), J1.B7 (D-)
- net GND: now also J1.A1 (GND), J1.A12 (GND), J1.B1 (GND), J1.B12 (GND), J1.S1 (SHIELD), R5.2, R6.2
- new net: J1.B5 (CC2), R5.1
- new net: J1.A5 (CC1), R6.1
- new net VCC: F2.1, J1.A4 (VBUS), J1.A9 (VBUS), J1.B4 (VBUS), J1.B9 (VBUS)

Commit message: completed schematic V1
Parts:
- added D1, D2, D3, D4: S0D-123, Diode_SMD:D_SOD-123, symbol Device:D_Small
- added MX1, MX2, MX3, MX4: MX-NoLED, MX_Alps_Hybrid:MX-1U, symbol MX_Alps_Hybrid:MX-NoLED
- C1, C2, C3, C4, C5, C6, C7: footprint (none) -> Capacitor_SMD:C_0805_2012Metric
- F2: footprint (none) -> Fuse:Fuse_1206_3216Metric
- J1: footprint (none) -> Connector_USB:USB_C_Receptacle_HRO_TYPE-C-31-M-12
- R1, R2, R3, R4, R5, R6: footprint (none) -> Resistor_SMD:R_0805_2012Metric
- SW1: footprint (none) -> random-keyboard-parts:SKQG-1155865
- Y1: footprint (none) -> Crystal:Crystal_SMD_3225-4Pin_3.2x2.5mm
Connections:
- new net: D1.2 (A), MX1.2 (ROW)
- new net: D4.2 (A), MX4.2 (ROW)
- new net: D3.2 (A), MX3.2 (ROW)
- new net: D2.2 (A), MX2.2 (ROW)
- new net Col0: MX1.1 (COL), MX3.1 (COL)
- new net Col1: MX2.1 (COL), MX4.1 (COL)
- new net Row0: D1.1 (K), D2.1 (K)
- new net Row1: D3.1 (K), D4.1 (K)
Other:
- moved on the sheet: C1, C2, C3, C4, C5, C6, C7, F2, J1, R1, R2, R3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
